File: atlas-flight-controller-board-v4/sd-card.kicad_sch (KiCad schematic)
At the start: 2 parts

Commit message: wip commit, hopefully last from mac
Parts:
- C28: footprint Capacitor_SMD:C_0603_1608Metric_Pad1.08x0.95mm_HandSolder -> Capacitor_SMD:C_0603_1608Metric
Connections:
- net CS_SD renamed CS_FLASH
- net MISO_SD renamed MISO_FLASH
- net MOSI_SD renamed MOSI_FLASH
- net SCK_SD renamed SCK_FLASH
Other:
- moved on the sheet: C28
Changed lines of the file:
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@@
 	(paper "A4")
 	(junction
-		(at 154.94 87.63)
+		(at 157.48 87.63)
 		(diameter 0)
 		(color 0 0 0 0)
@@
 	(wire
 		(pts
-			(xy 139.7 87.63) (xy 154.94 87.63)
+			(xy 139.7 87.63) (xy 157.48 87.63)
 		)
 		(stroke
@@
 	(wire
 		(pts
-			(xy 154.94 91.44) (xy 154.94 92.71)
+			(xy 157.48 91.44) (xy 157.48 92.71)
 		)
 		(stroke
@@
 	(wire
 		(pts
-			(xy 154.94 87.63) (xy 154.94 86.36)
+			(xy 157.48 87.63) (xy 157.48 86.36)
 		)
 		(stroke
@@
 		)
 	)
-	(global_label "MISO_SD"
+	(global_label "MISO_FLASH"
 		(shape input)
 		(at 139.7 92.71 0)
@@
 		)
 		(property "Intersheetrefs" "${INTERSHEET_REFS}"
-			(at 150.7285 92.71 0)
+			(at 153.9943 92.71 0)
 			(hide yes)
 			(show_name no)
@@
 		)
 	)
-	(global_label "CS_SD"
+	(global_label "CS_FLASH"
 		(shape input)
 		(at 119.38 90.17 180)
@@
 		)
 		(property "Intersheetrefs" "${INTERSHEET_REFS}"
-			(at 110.4682 90.17 0)
+			(at 107.2024 90.17 0)
 			(hide yes)
 			(show_name no)
@@
 		)
 	)
-	(global_label "MOSI_SD"
+	(global_label "MOSI_FLASH"
 		(shape input)
 		(at 139.7 95.25 0)
@@
 		)
 		(property "Intersheetrefs" "${INTERSHEET_REFS}"
-			(at 150.7285 95.25 0)
+			(at 153.9943 95.25 0)
 			(hide yes)
 			(show_name no)
@@
 		)
 	)
-	(global_label "SCK_SD"
+	(global_label "SCK_FLASH"
 		(shape input)
 		(at 119.38 92.71 180)
@@
 		)
 		(property "Intersheetrefs" "${INTERSHEET_REFS}"
-			(at 109.1982 92.71 0)
+			(at 105.9324 92.71 0)
 			(hide yes)
 			(show_name no)
@@
 	(symbol
 		(lib_id "Device:C_Small")
-		(at 154.94 90.17 0)
+		(at 157.48 90.17 0)
 		(unit 1)
 		(body_style 1)
@@
 		(fields_autoplaced yes)
 		(property "Reference" "C28"
-			(at 157.48 88.9062 0)
+			(at 160.02 88.9062 0)
 			(show_name no)
 			(do_not_autoplace no)
@@
 		)
 		(property "Value" "100 uF"
-			(at 157.48 91.4462 0)
+			(at 160.02 91.4462 0)
 			(show_name no)
 			(do_not_autoplace no)
@@
 			)
 		)
-		(property "Footprint" "Capacitor_SMD:C_0603_1608Metric_Pad1.08x0.95mm_HandSolder"
-			(at 154.94 90.17 0)
+		(property "Footprint" "Capacitor_SMD:C_0603_1608Metric"
+			(at 157.48 90.17 0)
 			(hide yes)
 			(show_name no)
@@
 		)
 		(property "Datasheet" ""
-			(at 154.94 90.17 0)
+			(at 157.48 90.17 0)
 			(hide yes)
 			(show_name no)
@@
 		)
 		(property "Description" "Unpolarized capacitor, small symbol"
-			(at 154.94 90.17 0)
+			(at 157.48 90.17 0)
 			(hide yes)
 			(show_name no)
@@
 	(symbol
 		(lib_id "power:GND")
-		(at 154.94 91.44 0)
+		(at 157.48 91.44 0)
 		(unit 1)
 		(body_style 1)
@@
 		(fields_autoplaced yes)
 		(property "Reference" "#PWR031"
-			(at 154.94 97.79 0)
+			(at 157.48 97.79 0)
 			(hide yes)
 			(show_name no)
@@
 		)
 		(property "Value" "GND"
-			(at 154.94 96.52 0)
+			(at 157.48 96.52 0)
 			(show_name no)
 			(do_not_autoplace no)
@@
 		)
 		(property "Footprint" ""
-			(at 154.94 91.44 0)
+			(at 157.48 91.44 0)
 			(hide yes)
 			(show_name no)
@@
 		)
 		(property "Datasheet" ""
-			(at 154.94 91.44 0)
+			(at 157.48 91.44 0)
 			(hide yes)
 			(show_name no)
@@
 		)
 		(property "Description" "Power symbol creates a global label with name \"GND\" , ground"
-			(at 154.94 91.44 0)
+			(at 157.48 91.44 0)
 			(hide yes)
 			(show_name no)
@@
 	(symbol
 		(lib_id "power:+3V3")
-		(at 154.94 86.36 0)
+		(at 157.48 86.36 0)
 		(unit 1)
 		(body_style 1)
@@
 		(fields_autoplaced yes)
 		(property "Reference" "#PWR030"
-			(at 154.94 90.17 0)
+			(at 157.48 90.17 0)
 			(hide yes)
 			(show_name no)
@@
 		)
 		(property "Value" "+3V3"
-			(at 154.94 81.28 0)
+			(at 157.48 81.28 0)
 			(show_name no)
 			(do_not_autoplace no)
@@
 		)
 		(property "Footprint" ""
-			(at 154.94 86.36 0)
+			(at 157.48 86.36 0)
 			(hide yes)
 			(show_name no)
@@
 		)
 		(property "Datasheet" ""
-			(at 154.94 86.36 0)
+			(at 157.48 86.36 0)
 			(hide yes)
 			(show_name no)
@@
 		)
 		(property "Description" "Power symbol creates a global label with name \"+3V3\""
-			(at 154.94 86.36 0)
-			(hide yes)
-			(show_name no)
+			(at 157.48 86.36 0)
+			(hide yes)
+			(show_name no)

Commit message: schematic done mostly besides style and footprints
Parts:
- removed C28: 100 uF, Capacitor_SMD:C_0603_1608Metric, symbol Device:C_Small
- removed U6: (no value), ZDSD16GLGIAG:LGA-8_8x6.2mm_P1.27mm, symbol sd-nand-flash:ZDSD16GLGIAG
Connections:
- no-connect marks 2 -> 0
Other:
- company: (none) -> Sam Manley, ARCUIA
- title: (none) -> Atlas v4 Flight Controller
