File: atlas-flight-controller-board-v4/atlas-flight-controller-board-v4.kicad_pcb (KiCad board)
At the start: 2 copper layers, 33.3 x 54.1 mm, 52 parts, among them IC1 LSM6DSV80XTR, J1 DX07S016JA1R1500, J2 Conn_Coaxial, J3 Conn_Coaxial, U1 STM32F405RGTx, U2 LIS2MDL, U3 SAM-M10Q-00B, U4 Value, U5 INA260, Y1 16 MHz

Commit message: wip commit, hopefully last from mac
Parts:
- removed C1: 10 uF, APA0606100M050R:CAP_APA_0606_AVX
- added C40: 100nF, Capacitor_SMD:C_0603_1608Metric, F.Cu at (101.1, 53.0)
- added C41: 1uF, Capacitor_SMD:C_0603_1608Metric, F.Cu at (132.7, 88.0)
- added C42: 1uF, Capacitor_SMD:C_0603_1608Metric, F.Cu at (133.1, 85.5)
- added C43: 10uF, Capacitor_SMD:C_0603_1608Metric, F.Cu at (120.4, 83.2)
- added C44: 100nF, Capacitor_SMD:C_0603_1608Metric, F.Cu at (120.0, 91.0)
- added C45: 100nF, Capacitor_SMD:C_0603_1608Metric, F.Cu at (123.2, 92.8)
- added FB3: 782853200, Inductor_SMD:L_0805_2012Metric, F.Cu at (66.2, 105.0)
- added FB4: 100R @ 100 MHz, Inductor_SMD:L_0603_1608Metric, F.Cu at (121.6, 91.0)
- added H1: MountingHole, MountingHole:MountingHole_2.2mm_M2_Pad_Via, F.Cu at (113.0, 43.0)
- added H2: MountingHole, MountingHole:MountingHole_2.2mm_M2_Pad_Via, F.Cu at (152.0, 43.0)
- added H3: MountingHole, MountingHole:MountingHole_2.2mm_M2_Pad_Via, F.Cu at (113.0, 97.0)
- added H4: MountingHole, MountingHole:MountingHole_2.2mm_M2_Pad_Via, F.Cu at (152.0, 97.0)
- added J2: Conn_Coaxial, Connector_Coaxial:SMA_Amphenol_132289_EdgeMount, B.Cu at (142.5, 42.5)
- added J3: Conn_Coaxial, Connector_Coaxial:SMA_Amphenol_132289_EdgeMount, B.Cu at (122.5, 42.5)
- added J4: Batt Conn, Connector_JST:JST_PH_S2B-PH-K_1x02_P2.00mm_Horizontal, F.Cu at (132.1, 93.5)
- added J5: Conn_ARM_SWD_TagConnect_TC2030-NL, Connector:Tag-Connect_TC2030-IDC-NL_2x03_P1.27mm_Vertical, F.Cu at (141.1, 89.0)
- added R16: ~, Resistor_SMD:R_0603_1608Metric, F.Cu at (131.2, 90.9)
- added R17: 10k, Resistor_SMD:R_0603_1608Metric, F.Cu at (101.3, 41.5)
- added R18: 10k, Resistor_SMD:R_0603_1608Metric, F.Cu at (101.1, 55.5)
- added R4: 33k, Resistor_SMD:R_0603_1608Metric, F.Cu at (95.6, 125.3)
- added R5: 82k, Resistor_SMD:R_0603_1608Metric, F.Cu at (93.2, 125.3)
- added R6: 5k1, Resistor_SMD:R_0603_1608Metric, F.Cu at (113.6, 82.6)
- added R7: 5k1, Resistor_SMD:R_0603_1608Metric, F.Cu at (116.8, 94.8)
- added R8: ~, Resistor_SMD:R_0603_1608Metric, F.Cu at (127.5, 88.9)
- added REF**: Molex_PicoBlade_53048-0610_1x06_P1.25mm_Horizontal, Connector_Molex:Molex_PicoBlade_53048-0610_1x06_P1.25mm_Horizontal, F.Cu at (138.6, 95.0)
- added U10: ~, Package_SON:WSON-8-1EP_2x2mm_P0.5mm_EP0.9x1.6mm, F.Cu at (131.1, 85.6)
- added U7: TPS62912, Package_DFN_QFN:Texas_RPU0010A_VQFN-HR-10_2x2mm_P0.5mm, F.Cu at (65.9, 102.6)
- added U8: TPS2116DRL, Package_TO_SOT_SMD:SOT-583-8, F.Cu at (129.8, 88.6)
- added U9: USBLC6, Package_TO_SOT_SMD:SOT-666, F.Cu at (119.4, 88.3)
- C10, C11, C12, C13, C14, C15, C16, C17, C18, C19, C20, C21, C22, C27, C28, C5, C6, C7, C8, C9: footprint Capacitor_SMD:C_0603_1608Metric_Pad1.08x0.95mm_HandSolder -> Capacitor_SMD:C_0603_1608Metric
- C2, C3: value 100 nF -> 100nF; footprint Capacitor_SMD:C_0603_1608Metric_Pad1.08x0.95mm_HandSolder -> Capacitor_SMD:C_0603_1608Metric
- C4: value 220 nF -> 220nF; footprint Capacitor_SMD:C_0603_1608Metric_Pad1.08x0.95mm_HandSolder -> Capacitor_SMD:C_0603_1608Metric
- R1: footprint Resistor_SMD:R_0603_1608Metric_Pad0.98x0.95mm_HandSolder -> Resistor_SMD:R_0603_1608Metric
- U2: footprint LIS2MDL:PQFN50P200X200X70-12N -> Package_LGA:LGA-12_2x2mm_P0.5mm
- Y1: footprint Crystal:Crystal_SMD_3225-4Pin_3.2x2.5mm_HandSoldering -> Crystal:Crystal_SMD_3225-4Pin_3.2x2.5mm
- moved R11 94.5 mm to (213.0, 57.6)
- moved R13 94.5 mm to (213.0, 60.1)
- moved R14 94.5 mm to (213.0, 61.4)
- moved C25 94.5 mm to (212.6, 48.4)
- moved R1 94.5 mm to (166.4, 18.9), turned to 90 degrees
- moved C26 94.5 mm to (212.6, 51.5)
- moved U4 94.5 mm to (221.9, 46.1)
- moved J2 94.4 mm to (229.3, 44.5)
- moved J3 94.4 mm to (213.0, 44.5)
- moved L2 94.4 mm to (213.0, 50.0)
- moved C24 94.4 mm to (229.6, 48.6)
- moved L1 94.4 mm to (229.3, 50.1)
- moved C29 94.4 mm to (211.2, 65.1)
- moved C30 94.4 mm to (213.3, 65.1)
- moved R10 94.4 mm to (213.0, 56.3)
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Connections:
- net /NRST renamed NRST
- net RAD_BUSY renamed BUSY_LORA
- net RAD_IRQ renamed IRQ_LORA
- net RAD_NSS renamed NSS_LORA
- net RAD_RESET renamed RST_LORA
- J1 pad 3: unconnected-(J1-CC1-Pad3) -> Net-(J1-CC1)
- J1 pad 5: Net-(J1-D--Pad5) -> /USB_DP-
- J1 pad 6: Net-(J1-D+-Pad6) -> /USB_DP+
- J1 pad 7: Net-(J1-D+-Pad6) -> /USB_DP+
- J1 pad 8: Net-(J1-D--Pad5) -> /USB_DP-
- J1 pad 9: unconnected-(J1-CC2-Pad9) -> Net-(J1-CC2)
- R11 pad 2: RAD_SCK -> SCK_LORA
- R12 pad 2: RAD_MOSI -> MOSI_LORA
- R13 pad 2: RAD_MISO -> MISO_LORA
- U1 pad 20: unconnected-(U1-PA4-Pad20) -> CS_LORA
- U1 pad 21: unconnected-(U1-PA5-Pad21) -> SCK_LORA
- U1 pad 22: unconnected-(U1-PA6-Pad22) -> MISO_LORA
- U1 pad 23: unconnected-(U1-PA7-Pad23) -> MOSI_LORA
- U1 pad 28: unconnected-(U1-PB2-Pad28) -> Net-(U1-PB2)
- U1 pad 34: unconnected-(U1-PB13-Pad34) -> SCK_MEMS
- U1 pad 35: unconnected-(U1-PB14-Pad35) -> MISO_MEMS
- U1 pad 36: unconnected-(U1-PB15-Pad36) -> MOSI_MEMS
- U1 pad 42: unconnected-(U1-PA9-Pad42) -> /VBUS_SENSE
- U1 pad 44: unconnected-(U1-PA11-Pad44) -> /USB_DP-
- U1 pad 45: unconnected-(U1-PA12-Pad45) -> /USB_DP+
- U1 pad 46: /SWDIO -> SWDIO
- U1 pad 49: /SWCLK -> SWCLK
- U1 pad 51: unconnected-(U1-PC10-Pad51) -> FLASH_SCK
- U1 pad 52: unconnected-(U1-PC11-Pad52) -> FLASH_MISO
- U1 pad 53: unconnected-(U1-PC12-Pad53) -> FLASH_MOSI
- U1 pad 55: unconnected-(U1-PB3-Pad55) -> SWO
Routing:
- net Net-(J1-CC1): track 0.00 -> 5.57 mm
- net /USB_DP-: track 0.00 -> 4.62 mm
- net /USB_DP+: track 0.00 -> 2.25 mm
Other:
- board size 33.3 x 54.1 mm -> 127.6 x 60 mm
- copper layers 2 -> 4
- board text added: "NEED TO IMPEDANCE MATCH USB. Check thickness and routing off power"

Commit message: schematic done mostly besides style and footprints
Parts:
- removed the C11 at (162.0, 22.2)
- removed the C12 at (157.4, 25.2)
- removed the C13 at (160.5, 25.2)
- removed the C14 at (157.4, 19.1)
- removed the C15 at (160.5, 19.1)
- removed the C16 at (157.4, 22.2)
- removed the C17 at (159.0, 25.2)
- removed C18: 1 uF, Capacitor_SMD:C_0603_1608Metric
- removed the C19 at (159.0, 22.2)
- removed C20: 100 nF, Capacitor_SMD:C_0603_1608Metric
- removed C21, C22: 10 pF, Capacitor_SMD:C_0603_1608Metric
- removed C28: 100 uF, Capacitor_SMD:C_0603_1608Metric
- removed the J1 at (115.7, 88.5)
- removed the R1 at (166.4, 18.9)
- removed the R4 at (95.6, 125.3)
- removed the R5 at (93.2, 125.3)
- removed REF**: Molex_PicoBlade_53048-0610_1x06_P1.25mm_Horizontal, Connector_Molex:Molex_PicoBlade_53048-0610_1x06_P1.25mm_Horizontal
- removed the U1 at (132.6, 75.0)
- removed the U6 at (150.1, 86.2)
- added C31: 4u7, Capacitor_SMD:C_0805_2012Metric, F.Cu at (106.5, 50.0)
- added C32: 100 nF, Capacitor_SMD:C_0603_1608Metric, F.Cu at (94.3, 49.7)
- added C33: 100n, Capacitor_SMD:C_0603_1608Metric, F.Cu at (94.3, 52.2)
- added C34: 10 pF, Capacitor_SMD:C_0603_1608Metric, F.Cu at (142.0, 65.0)
- added C35: 100 nF, Capacitor_SMD:C_0603_1608Metric, F.Cu at (94.3, 54.8)
- added C36: 100 nF, Capacitor_SMD:C_0603_1608Metric, F.Cu at (94.3, 57.3)
- added C37: 10 pF, Capacitor_SMD:C_0603_1608Metric, F.Cu at (142.0, 63.5)
- added C38: 100 nF, Capacitor_SMD:C_0603_1608Metric, F.Cu at (94.3, 59.8)
- added C39: 100 nF, Capacitor_SMD:C_0603_1608Metric, F.Cu at (94.3, 62.3)
- added C41: 100 uF, Capacitor_SMD:C_0603_1608Metric, F.Cu at (98.3, 52.2)
- added C42: 1 uF, Capacitor_SMD:C_0603_1608Metric, F.Cu at (98.3, 54.8)
- added C43: 1 uF, Capacitor_SMD:C_0603_1608Metric, F.Cu at (98.3, 57.3)
- added C44: 100nF, Capacitor_SMD:C_0603_1608Metric, F.Cu at (98.3, 59.8)
- added C45: 100nF, Capacitor_SMD:C_0603_1608Metric, F.Cu at (105.2, 67.2)
- added C46: 10n, Capacitor_SMD:C_0603_1608Metric, F.Cu at (147.0, 58.5)
- added C47: 10n, Capacitor_SMD:C_0603_1608Metric, F.Cu at (147.0, 64.0)
- added C48: 10u, Capacitor_SMD:C_0805_2012Metric, F.Cu at (143.1, 77.2)
- added C49: 10n, Capacitor_SMD:C_0603_1608Metric, F.Cu at (147.0, 69.0)
- added C50: 100nF, Capacitor_SMD:C_0603_1608Metric, F.Cu at (103.2, 100.6)
- added C51: 2u2, Capacitor_SMD:C_0603_1608Metric, F.Cu at (94.0, 41.3)
- added C52: 2u2, Capacitor_SMD:C_0603_1608Metric, F.Cu at (94.0, 43.8)
- added D14: LED-Red, LED_SMD:LED_0402_1005Metric, F.Cu at (145.0, 56.0)
- added D15: LED-Red, LED_SMD:LED_0402_1005Metric, F.Cu at (145.0, 61.5)
- added D16: LED-Red, LED_SMD:LED_0402_1005Metric, F.Cu at (145.0, 66.5)
- added D17: LED-Red, LED_SMD:LED_0402_1005Metric, F.Cu at (97.2, 67.0)
- added D18: LED-Red, LED_SMD:LED_0402_1005Metric, F.Cu at (97.2, 69.0)
- added D19: LED-Red, LED_SMD:LED_0402_1005Metric, F.Cu at (97.2, 71.0)
- added J4: DX07S016JA1R1500, usb-c:JAE_DX07S016JA1R1500, F.Cu at (122.0, 95.0)
- added J6: Screw_Terminal_01x06, TerminalBlock:TerminalBlock_Xinya_XY308-2.54-6P_1x06_P2.54mm_Horizontal, F.Cu at (151.5, 70.0)
- added J7: Conn_01x02, Connector_JST:JST_PH_S2B-PH-K_1x02_P2.00mm_Horizontal, F.Cu at (148.6, 77.0)
- added J8: Conn_01x08, Connector_Molex:Molex_PicoBlade_53048-0810_1x08_P1.25mm_Horizontal, F.Cu at (138.1, 95.3)
- added Q12: BSS138, Package_TO_SOT_SMD:SOT-23, F.Cu at (95.0, 96.6)
- added R10: 15k4, Resistor_SMD:R_0402_1005Metric, F.Cu at (99.5, 41.0)
- added R11: 4k87, Resistor_SMD:R_0402_1005Metric, F.Cu at (99.5, 43.0)
- added R16: 10k, Resistor_SMD:R_0603_1608Metric, F.Cu at (98.3, 62.3)
- added R19: 33k, Resistor_SMD:R_0402_1005Metric, F.Cu at (102.3, 52.2)
- added R20: 5k1, Resistor_SMD:R_0603_1608Metric, F.Cu at (102.3, 54.8)
- added R21: 5k1, Resistor_SMD:R_0603_1608Metric, F.Cu at (102.3, 57.3)
- added R22: 10k, Resistor_SMD:R_0603_1608Metric, F.Cu at (102.3, 59.8)
- added R24: 10k, Resistor_SMD:R_0603_1608Metric, F.Cu at (105.7, 100.6)
- added R26: 10k, Resistor_SMD:R_0603_1608Metric, B.Cu at (208.0, 55.2)
- added R27: 100k, Resistor_SMD:R_0603_1608Metric, F.Cu at (105.2, 72.2)
- added R32: 15k, Resistor_SMD:R_0603_1608Metric, F.Cu at (145.0, 58.5)
- added R33: 15k, Resistor_SMD:R_0603_1608Metric, F.Cu at (159.0, 73.0)
- added R34: 15k, Resistor_SMD:R_0603_1608Metric, F.Cu at (159.0, 75.5)
- added R35: 15k, Resistor_SMD:R_0603_1608Metric, F.Cu at (159.0, 78.0)
- added R36: 1k5, Resistor_SMD:R_0603_1608Metric, F.Cu at (93.5, 67.2)
- added R37: 15k, Resistor_SMD:R_0603_1608Metric, F.Cu at (145.0, 64.0)
- added R38: 15k, Resistor_SMD:R_0603_1608Metric, F.Cu at (145.0, 69.0)
- added R39: 1k5, Resistor_SMD:R_0603_1608Metric, F.Cu at (93.5, 69.8)
- added R40: 1k5, Resistor_SMD:R_0603_1608Metric, F.Cu at (93.5, 72.3)
- added R41: 1k5, Resistor_SMD:R_0603_1608Metric, F.Cu at (98.5, 97.0)
- added R43: 330, PCM_SparkFun-Resistor:R_0603_1608Metric, F.Cu at (158.0, 68.8)
- added R44: 330, PCM_SparkFun-Resistor:R_0603_1608Metric, F.Cu at (93.5, 76.8)
- added SW3: SW_Push, myButtons:SW_USLPT2819DT2TR, F.Cu at (94.2, 88.8)
- added SW4: HARD_RESET, myButtons:SW_USLPT2819DT2TR, F.Cu at (94.2, 83.4)
- added TP1: TestPoint_Square, TestPoint:TestPoint_Pad_2.0x2.0mm, F.Cu at (161.0, 92.5)
- added TP11: TestPoint_Square, TestPoint:TestPoint_Pad_1.5x1.5mm, F.Cu at (94.6, 100.8)
- added TP12: TestPoint_Square, TestPoint:TestPoint_Pad_1.5x1.5mm, F.Cu at (98.2, 100.8)
- added TP2: TestPoint_Square, TestPoint:TestPoint_Pad_2.0x2.0mm, F.Cu at (161.0, 96.6)
- added TP3: TestPoint_Square, TestPoint:TestPoint_Pad_2.0x2.0mm, F.Cu at (165.5, 92.5)
- added TP4: TestPoint_Square, TestPoint:TestPoint_Pad_2.0x2.0mm, F.Cu at (165.5, 96.6)
- added TP5: TestPoint_Square, TestPoint:TestPoint_Pad_2.0x2.0mm, F.Cu at (172.5, 84.5)
- added TP6: TestPoint_Square, TestPoint:TestPoint_Pad_2.0x2.0mm, F.Cu at (172.5, 88.6)
- added TP7: TestPoint_Square, TestPoint:TestPoint_Pad_2.0x2.0mm, F.Cu at (172.5, 92.6)
- added TP8: TestPoint_Square, TestPoint:TestPoint_Pad_2.0x2.0mm, F.Cu at (172.5, 96.7)
- added U10: USBLC6, Package_TO_SOT_SMD:SOT-666, F.Cu at (122.0, 91.0)
- added U11: VNQ7140AJTR, VNQ7140AJTR:SOIC_0AJTR_STM, F.Cu at (143.0, 73.5)
- added U8: STM32F405RGTx, Package_QFP:LQFP-64_10x10mm_P0.5mm, F.Cu at (130.0, 74.0)
- C1: renamed from C5; footprint Capacitor_SMD:C_0603_1608Metric -> Capacitor_SMD:C_0402_1005Metric
- C10: renamed from C8; footprint Capacitor_SMD:C_0603_1608Metric -> Capacitor_SMD:C_0402_1005Metric
- C11: renamed from C10; footprint Capacitor_SMD:C_0603_1608Metric -> Capacitor_SMD:C_0402_1005Metric
- C14: renamed from C29; value 100 uF -> 100n; footprint Capacitor_SMD:C_0603_1608Metric_Pad1.08x0.95mm_HandSolder -> Resistor_SMD:R_0603_1608Metric
- C15: renamed from C30; value 10 uF -> 10u; footprint Capacitor_SMD:C_0603_1608Metric_Pad1.08x0.95mm_HandSolder -> Resistor_SMD:R_0603_1608Metric
- C3: renamed from C2; footprint Capacitor_SMD:C_0603_1608Metric -> Capacitor_SMD:C_0402_1005Metric
- C4: renamed from C3; footprint Capacitor_SMD:C_0603_1608Metric -> Capacitor_SMD:C_0402_1005Metric
- C40: value 100nF -> 10 nF
- C5: renamed from C4; footprint Capacitor_SMD:C_0603_1608Metric -> Capacitor_SMD:C_0402_1005Metric
- C6: footprint Capacitor_SMD:C_0603_1608Metric -> Capacitor_SMD:C_0402_1005Metric
- C7: renamed from C27; footprint Capacitor_SMD:C_0603_1608Metric -> Capacitor_SMD:C_0402_1005Metric
- C8: renamed from C9; footprint Capacitor_SMD:C_0603_1608Metric -> Capacitor_SMD:C_0402_1005Metric
- C9: renamed from C7; footprint Capacitor_SMD:C_0603_1608Metric -> Capacitor_SMD:C_0402_1005Metric
- J5: value Conn_ARM_SWD_TagConnect_TC2030-NL -> SWD_TC2030-NL
- R17: value 10k -> 33k
- R18: value 10k -> 82k; footprint Resistor_SMD:R_0603_1608Metric -> Resistor_SMD:R_0402_1005Metric
- R8: value ~ -> 100k; footprint Resistor_SMD:R_0603_1608Metric -> Resistor_SMD:R_0402_1005Metric
- R9: renamed from R16; value ~ -> 33k
- U7: renamed from U10; value ~ -> TPS7A2133PQWDSGRQ1
- U9: value USBLC6 -> ~; footprint Package_TO_SOT_SMD:SOT-666 -> ZDSD16GLGIAG:LGA-8_8x6.2mm_P1.27mm
- moved U9 29.6 mm to (149.0, 88.5), turned to 90 degrees
- moved R17 28.5 mm to (105.2, 69.7)
- moved C19 17.3 mm to (103.0, 88.0)
- moved FB2 16.5 mm to (105.5, 87.3), turned to 0 degrees
- moved C23 16.0 mm to (108.0, 87.8)
- moved R7 15.5 mm to (106.7, 83.0)
- moved R6 10.8 mm to (102.8, 83.1)
- moved C4 9.23 mm to (117.8, 87.0), turned to 90 degrees
- moved C1 8.77 mm to (112.5, 77.5)
- moved IC1 8.38 mm to (115.2, 78.2)
- moved C5 8.24 mm to (114.0, 85.8)
- moved Y1 8.21 mm to (142.0, 68.0)
- moved U1 7.84 mm to (115.8, 85.8)
- moved C6 7.77 mm to (112.5, 79.5)
- moved C9 7.63 mm to (112.5, 82.5)
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- renumbered C24 to C12, C23 to C13, C26 to C16, C25 to C17, C44 to C19, C43 to C2, C45 to C23, C41 to C27, C42 to C29, FB4 to FB2, J2 to J1, J3 to J2, J4 to J3, R15 to R1, R9 to R2, R10 to R3, R11 to R4, R12 to R5, R13 to R6, R14 to R7, U2 to U1, U5 to U2, U7 to U5, U8 to U6
Connections:
- C12 pad 1: Net-(J2-In) -> Net-(J1-In)
- C17 pad 1: Net-(J3-In) -> Net-(J2-In)
- C40 pad 1: GND -> +3.3VA
- C40 pad 2: Net-(C40-Pad2) -> GND
- J1 pad 1: Net-(J2-In) -> Net-(J1-In)
- J2 pad 1: Net-(J3-In) -> Net-(J2-In)
- J3 pad 2: Net-(J4-Pin_2) -> /power/VBATT+
- L1 pad 1: Net-(J2-In) -> Net-(J1-In)
- L2 pad 1: Net-(J3-In) -> Net-(J2-In)
- R17 pad 1: Net-(U1-PB2) -> /power/VBATT+
- R17 pad 2: /SW_BOOT1 -> BATT_SENSE
- R18 pad 1: STANDBY_TOGGLE -> GND
- R18 pad 2: Net-(C40-Pad2) -> /stm32/VBUS_SENSE
- U6 pad 6: Net-(J4-Pin_2) -> /power/VBATT+
- U7 pad 2: GND -> Net-(U7-Pad2)
- U7 pad 3: GND -> Net-(U7-Pad2)
- U7 pad 5: /power/MUX OUT -> Net-(U7-EN)
- U7 pad 6: GND -> Net-(U7-Pad2)
- U7 pad 7: GND -> Net-(U7-Pad2)
- U9 pad 1: /USB_DP- -> unconnected-(U9-XX-Pad1)
- U9 pad 2: GND -> CS_FLASH
- U9 pad 3: /USB_DP+ -> SCK_FLASH
- U9 pad 4: /USB_DP+ -> GND
- U9 pad 5: VBUS -> MOSI_FLASH
- U9 pad 6: /USB_DP- -> MISO_FLASH
- Y1 pad 1: /HSE_IN -> /stm32/HSE_IN
- Y1 pad 3: /HSE_OUT -> /stm32/HSE_OUT
Routing:
- net GND: track 0.00 -> 10.8 mm, vias 0 -> 1
- net +3V3: track 0.00 -> 10.8 mm
- net Net-(J1-CC1): track 5.57 -> 0.00 mm
- net Net-(J1-In): track 0.00 -> 5.10 mm
- net Net-(J2-In): track 0.00 -> 4.98 mm
- net /USB_DP-: track 4.62 -> 0.00 mm
- net Net-(U4-Sub-G_RF): track 0.00 -> 4.11 mm
- net Net-(U4-2.4G_RF): track 0.00 -> 4.00 mm
- net <NO NET>: track 0.00 -> 2.68 mm
- net /USB_DP+: track 2.25 -> 0.00 mm
- net Net-(U1-C1): track 0.00 -> 1.17 mm
- net Net-(J6-Pin_5): track 0.00 -> 1.16 mm
- net Net-(J6-Pin_3): track 0.00 -> 0.57 mm
