File: atlas-flight-controller-board-v4/power.kicad_sch (KiCad schematic)
At the start: 14 parts, among them U7 TPS62913

Commit message: wip commit, hopefully last from mac
Parts:
- added C41, C42: 1uF, Capacitor_SMD:C_0603_1608Metric, symbol Device:C_Small
- added C44, C45: 100nF, Capacitor_SMD:C_0603_1608Metric, symbol Device:C_Small
- added FB4: 100R @ 100 MHz, Inductor_SMD:L_0603_1608Metric, symbol Device:FerriteBead_Small
- added J4: Batt Conn, Connector_JST:JST_PH_S2B-PH-K_1x02_P2.00mm_Horizontal, symbol Connector_Generic:Conn_01x02
- added R16, R8: (no value), Resistor_SMD:R_0603_1608Metric, symbol Device:R_Small
- added U10: (no value), Package_SON:WSON-8-1EP_2x2mm_P0.5mm_EP0.9x1.6mm, symbol TPS7A12133PQWDSGRQ1:TPS7A2133PQWDSGRQ1
- added U8: TPS2116DRL, Package_TO_SOT_SMD:SOT-583-8, symbol Power_Management:TPS2116DRL
- FB3: value FerriteBead_Small -> 782853200; footprint (none) -> Inductor_SMD:L_0805_2012Metric
- U7: value TPS62913 -> TPS62912
Connections:
- net +3V3: now also C42.1, U10.1 (OUT); no longer C31.1, C32.1, C33.1, C38.1, C39.1, FB3.2, R2.1, U7.1 (EN/SYNC), U7.10 (S-CONF), U7.6 (VIN)
- net GND: now also C41.2, C42.2, C44.2, C45.2, J4.1 (Pin_1), R16.2, U10.2, U10.3, U10.4 (GND), U10.6, U10.7, U10.9 (PAD), U8.1 (GND)
- new net: C45.1, FB4.2, R8.1, U8.3 (VIN1), U8.5 (MODE)
- new net: R16.1, R8.2, U8.4 (PR1)
- new net: J4.2 (Pin_2), U8.6 (VIN2)
- new net +3V7: C38.1, C39.1, FB3.2, R2.1
- new net MUX OUT: C41.1, U10.5 (EN), U10.8 (IN), U8.2 (VOUT), U8.7 (VOUT)
- new net VBAT_OUT: C31.1, C32.1, C33.1, U7.1 (EN/SYNC), U7.10 (S-CONF), U7.6 (VIN)
- new net VBUS: C44.1, FB4.1
- no-connect marks 1 -> 2
Other:
- note added: "CHECK THESE VALUES AGAINST ONLINE CALCULATOR TO MAKE IT (3v3 + Vdrop)"
- note added: "EXTERNAL PYRO CIRCUTRY (DNP ON ATLAS)"
- note added: "THIS IS EXTERNAL, ON THE CONNECTOR BOARD (IF APPLICABLE)"
- note added: "This is VBATT after current sensor."
- note added: "just read in on gpio if vbus is high"
- moved on the sheet: C31, C32, C33, C34, C35, C36, C37, C38, C39, FB3, L3, R2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

Commit message: schematic done mostly besides style and footprints
Parts:
- added C22, C23: 100nF, Capacitor_SMD:C_0603_1608Metric, symbol Device:C_Small
- added C24: 10u, Capacitor_SMD:C_0805_2012Metric, symbol Device:C_Small
- added C25, C26, C27: 10n, Capacitor_SMD:C_0603_1608Metric, symbol Device:C_Small
- added D1, D2, D3: LED-Red, LED_SMD:LED_0402_1005Metric, symbol Device:LED
- added J4: Conn_01x02, Connector_JST:JST_PH_S2B-PH-K_1x02_P2.00mm_Horizontal, symbol Connector_Generic:Conn_01x02
- added J5: Screw_Terminal_01x06, TerminalBlock:TerminalBlock_Xinya_XY308-2.54-6P_1x06_P2.54mm_Horizontal, symbol Connector:Screw_Terminal_01x06
- added R11: 10k, Resistor_SMD:R_0402_1005Metric, symbol Device:R_Small
- added R12: 33k, Resistor_SMD:R_0402_1005Metric, symbol Device:R_Small
- added R13: 100k, Resistor_SMD:R_0402_1005Metric, symbol Device:R_Small
- added R14, R15, R16, R17, R18, R19: 15k, Resistor_SMD:R_0402_1005Metric, symbol Device:R_Small
- added R20, R21: 330, Resistor_SMD:R_0402_1005Metric, symbol Device:R_Small
- added SW1: HARD_RESET, myButtons:SW_USLPT2819DT2TR, symbol Switch:SW_Push
- added U10: VNQ7140AJTR, VNQ7140AJTR:SOIC_0AJTR_STM, symbol VNQ7140AJTR:VNQ7140AJTR
- C31: renamed from C33; now not fitted; now left out of the parts list
- R10: renamed from R16; value (none) -> 33k; footprint Resistor_SMD:R_0603_1608Metric -> Resistor_SMD:R_0402_1005Metric
- R22: renamed from R2; footprint (none) -> Resistor_SMD:R_0402_1005Metric
- R23: renamed from R3; footprint (none) -> Resistor_SMD:R_0402_1005Metric
- R9: renamed from R8; value (none) -> 100k; footprint Resistor_SMD:R_0603_1608Metric -> Resistor_SMD:R_0402_1005Metric
- U5: renamed from U10; value (none) -> TPS7A2133PQWDSGRQ1
- renumbered C44 to C18, C45 to C19, C42 to C20, C41 to C21, C34 to C28, C35 to C29, C36 to C30, C31 to C33, C38 to C34, C39 to C35, C37 to C36, FB4 to FB2, J4 to J3, U7 to U11, U8 to U6
Connections:
- net +3V3: now also U10.2 (SEN)
- net GND: now also C22.2, C23.1, C24.2, C25.2, C26.2, C27.2, J4.2 (Pin_2), J5.2 (Pin_2), J5.4 (Pin_4), J5.6 (Pin_6), R13.2, R17.2, R18.2, R19.2, R21.2, SW1.2, U10.10 (SEL2), U10.14 (INPUT3), U10.4 (GND); no longer U5.2, U5.3, U5.6, U5.7
- net MUX OUT: now also R11.2; no longer U5.5 (EN)
- net VBATT+: now reaches J3.2 (Pin_2), U6.6 (VIN2)
- net VBATT+: now also R12.1
- new net: C27.1, J5.1 (Pin_1), R16.2, U10.1 (OUTPUT0)
- new net: C23.2, R11.1, SW1.1, U5.5 (EN)
- new net: D3.1 (K), R16.1
- new net: D1.2 (A), D2.2 (A), D3.2 (A)
- new net: D2.1 (K), R15.1
- new net: C24.1, J4.1 (Pin_1)
- new net: R20.1, U10.13 (MULTISENSE)
- new net: C26.1, J5.3 (Pin_3), R15.2, U10.8 (OUTPUT1)
- new net: C25.1, J5.5 (Pin_5), R14.2, U10.9 (OUTPUT2)
- new net: D1.1 (K), R14.1
- new net: U10.17 (VCC), U10.5 (FAULTRS_T)
- new net: U5.2, U5.3, U5.6, U5.7
- new net BATT_SENSE: C22.1, R12.2, R13.1
- new net PYRO_1: R19.1, U10.3 (INPUT0)
- new net PYRO_2: R18.1, U10.6 (INPUT1)
- new net PYRO_3: R17.1, U10.11 (INPUT2)
- new net PYRO_MULTISENSE: R20.2, R21.1
- new net PYRO_SEL0: U10.12 (SEL0)
- new net PYRO_SEL1: U10.15 (SEL1)
- no-connect marks 2 -> 3
Other:
- note added: "EXTERNAL PYRO CIRCUTRY"
- note added: "NEEDS TO BE 1/2S. CANNOT BE HIGHER. CONTINUITY CURRENT WILL RISE"
- note added: "OUTPUTS 5V HIGH ON FAULT. R_SENSE = 660 I_SENSE_MAX = 4mA"
- note added: "need pd resistors prevent firing during mcu set up"
- note removed: "EXTERNAL PYRO CIRCUTRY (DNP ON ATLAS)"
- company: (none) -> Sam Manley, ARCUIA
- title: (none) -> Atlas v4 Flight Controller
- moved on the sheet: C18, C19, C20, C21, C28, C29, C30, C32, C33, C34, C35, C36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

Commit message: progress update. schematic has been done, layout is half finished. board is now 50x65mm for rf performance reasons
Parts:
- C34: renamed from C18; value 100nF -> 100n; footprint Capacitor_SMD:C_0603_1608Metric -> Capacitor_SMD:C_0402_1005Metric
- C35: renamed from C19; value 100nF -> 100n; footprint Capacitor_SMD:C_0603_1608Metric -> Capacitor_SMD:C_0402_1005Metric
- C36: renamed from C20; value 1uF -> 1u
- C37: renamed from C21; value 1uF -> 1u
- C38: renamed from C22; value 100nF -> 100n; footprint Capacitor_SMD:C_0603_1608Metric -> Capacitor_SMD:C_0402_1005Metric
- C39: renamed from C23; value 100nF -> 100n; footprint Capacitor_SMD:C_0603_1608Metric -> Capacitor_SMD:C_0402_1005Metric
- C41: renamed from C25; footprint Capacitor_SMD:C_0603_1608Metric -> Capacitor_SMD:C_0402_1005Metric
- C42: renamed from C26; footprint Capacitor_SMD:C_0603_1608Metric -> Capacitor_SMD:C_0402_1005Metric
- C43: renamed from C27; footprint Capacitor_SMD:C_0603_1608Metric -> Capacitor_SMD:C_0402_1005Metric
- C44: renamed from C28; value 22uF -> 22u
- C45: renamed from C29; value 22uF -> 22u
- C46: renamed from C30; value 22uF -> 22u
- C47: renamed from C31; value 10uF -> 10u; now fitted; now in the parts list
- C48: renamed from C32; value 10uF -> 10u
- C49: renamed from C33; value 22nF -> 22n
- C50: renamed from C34; value 22uF -> 22u
- C51: renamed from C35; value 22uF -> 22u
- C52: renamed from C36; value 470nF -> 470n
- FB3: renamed from FB2; value 100R @ 100 MHz -> 120R @ 100 MHz; footprint Inductor_SMD:L_0603_1608Metric -> Inductor_SMD:L_0402_1005Metric
- L3: value 22uH -> 22u
- R32: renamed from R22; footprint Resistor_SMD:R_0402_1005Metric -> (none)
- R33: renamed from R23; footprint Resistor_SMD:R_0402_1005Metric -> (none)
- renumbered C24 to C40, D1 to D5, D2 to D6, D3 to D7, FB3 to FB4, J3 to J6, J4 to J7, J5 to J8, R9 to R19, R10 to R20, R11 to R21, R12 to R22, R13 to R23, R14 to R24, R15 to R25, R16 to R26, R17 to R27, R18 to R28, R19 to R29, R20 to R30, R21 to R31, SW1 to SW3, U10 to U13, U11 to U14, U5 to U8, U6 to U9
Connections:
- net PYRO_BATT: now reaches D5.2 (A), D6.2 (A), D7.2 (A)
- net PYRO_BATT: now also C40.1, J7.1 (Pin_1), U13.17 (VCC), U13.5 (FAULTRS_T)
