File: atlas-flight-controller-board-v4/radio.kicad_sch (KiCad schematic)
At the start: 19 parts, among them J2 Conn_Coaxial, J3 Conn_Coaxial, U4 Value

Commit message: wip commit, hopefully last from mac
Connections:
- net RAD_BUSY renamed BUSY_LORA
- net RAD_IRQ renamed IRQ_LORA
- net RAD_MISO renamed MISO_LORA
- net RAD_MOSI renamed MOSI_LORA
- net RAD_NSS renamed NSS_LORA
- net RAD_RESET renamed RST_LORA
- net RAD_SCK renamed SCK_LORA
Changed lines of the file:
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@@
 		)
 	)
-	(global_label "RAD_NSS"
+	(global_label "NSS_LORA"
 		(shape input)
 		(at 157.48 90.17 0)
@@
 		)
 		(property "Intersheetrefs" "${INTERSHEET_REFS}"
-			(at 168.8109 90.17 0)
+			(at 169.8995 90.17 0)
 			(hide yes)
 			(show_name no)
@@
 		)
 	)
-	(global_label "RAD_IRQ"
+	(global_label "IRQ_LORA"
 		(shape input)
 		(at 116.84 95.25 180)
@@
 		)
 		(property "Intersheetrefs" "${INTERSHEET_REFS}"
-			(at 106.0533 95.25 0)
+			(at 104.9647 95.25 0)
 			(hide yes)
 			(show_name no)
@@
 		)
 	)
-	(global_label "RAD_MOSI"
+	(global_label "MOSI_LORA"
 		(shape input)
 		(at 157.48 95.25 0)
@@
 		)
 		(property "Intersheetrefs" "${INTERSHEET_REFS}"
-			(at 169.6576 95.25 0)
+			(at 170.7462 95.25 0)
 			(hide yes)
 			(show_name no)
@@
 		)
 	)
-	(global_label "RAD_SCK"
+	(global_label "SCK_LORA"
 		(shape input)
 		(at 157.48 92.71 0)
@@
 		)
 		(property "Intersheetrefs" "${INTERSHEET_REFS}"
-			(at 168.8109 92.71 0)
+			(at 169.8995 92.71 0)
 			(hide yes)
 			(show_name no)
@@
 		)
 	)
-	(global_label "RAD_MISO"
+	(global_label "MISO_LORA"
 		(shape input)
 		(at 157.48 97.79 0)
@@
 		)
 		(property "Intersheetrefs" "${INTERSHEET_REFS}"
-			(at 169.6576 97.79 0)
+			(at 170.7462 97.79 0)
 			(hide yes)
 			(show_name no)
@@
 		)
 	)
-	(global_label "RAD_RESET"
+	(global_label "RST_LORA"
 		(shape input)
 		(at 157.48 100.33 0)
@@
 		)
 		(property "Intersheetrefs" "${INTERSHEET_REFS}"
-			(at 170.8065 100.33 0)
+			(at 169.5971 100.33 0)
 			(hide yes)
 			(show_name no)
@@
 		)
 	)
-	(global_label "RAD_BUSY"
+	(global_label "BUSY_LORA"
 		(shape input)
 		(at 157.48 87.63 0)
@@
 		)
 		(property "Intersheetrefs" "${INTERSHEET_REFS}"
-			(at 169.96 87.63 0)
+			(at 171.0486 87.63 0)
 			(hide yes)
 			(show_name no)
@@
 		)
 	)
-	(group "ZDSD16GLGEAG_SPI"
-		(lib_id "nvm:ZDSD16GLGEAG_SPI")
-		(members "827bb21e-e577-4094-b64e-072da7c99db6" "c6d669ca-d717-41c6-b628-e5e3fb90d829"
-			"ecb4ec6f-689d-4abd-9e2b-0bd1476448c3"
-		)
-	)

Commit message: schematic done mostly besides style and footprints
Parts:
- added R8: 10k, Resistor_SMD:R_0402_1005Metric, symbol Device:R_Small
- C16: renamed from C29; value 100 uF -> 100n; footprint Capacitor_SMD:C_0603_1608Metric_Pad1.08x0.95mm_HandSolder -> Resistor_SMD:R_0603_1608Metric
- C17: renamed from C30; value 10 uF -> 10u; footprint Capacitor_SMD:C_0603_1608Metric_Pad1.08x0.95mm_HandSolder -> Resistor_SMD:R_0603_1608Metric
- renumbered C24 to C12, C23 to C13, C26 to C14, C25 to C15, FB2 to FB1, J2 to J1, J3 to J2, R9 to R1, R10 to R2, R11 to R3, R15 to R4, R12 to R5, R13 to R6, R14 to R7
Connections:
- net +3V3: now also R8.1
- net BUSY_LORA: now also R8.2
Other:
- company: (none) -> Sam Manley, ARCUIA
- title: (none) -> Atlas v4 Flight Controller

Commit message: progress update. schematic has been done, layout is half finished. board is now 50x65mm for rf performance reasons
Parts:
- removed FB1: FerriteBead_Small, symbol Device:FerriteBead_Small
- added FB2: 120R @ 100 MHz, Inductor_SMD:L_0402_1005Metric, symbol Device:FerriteBead_Small
- C32: renamed from C16; footprint Resistor_SMD:R_0603_1608Metric -> Capacitor_SMD:C_0402_1005Metric
- C33: renamed from C17; footprint Resistor_SMD:R_0603_1608Metric -> Capacitor_SMD:C_0603_1608Metric
- R11: renamed from R1; footprint Capacitor_SMD:C_0402_1005Metric_Pad0.74x0.62mm_HandSolder -> Resistor_SMD:R_0402_1005Metric
- R12: renamed from R2; footprint Capacitor_SMD:C_0402_1005Metric_Pad0.74x0.62mm_HandSolder -> Resistor_SMD:R_0402_1005Metric
- R13: renamed from R3; footprint Capacitor_SMD:C_0402_1005Metric_Pad0.74x0.62mm_HandSolder -> Resistor_SMD:R_0402_1005Metric
- R14: renamed from R4; footprint Capacitor_SMD:C_0402_1005Metric_Pad0.74x0.62mm_HandSolder -> Resistor_SMD:R_0402_1005Metric
- R15: renamed from R5; footprint Capacitor_SMD:C_0402_1005Metric_Pad0.74x0.62mm_HandSolder -> Resistor_SMD:R_0402_1005Metric
- R16: renamed from R6; footprint Capacitor_SMD:C_0402_1005Metric_Pad0.74x0.62mm_HandSolder -> Resistor_SMD:R_0402_1005Metric
- R17: renamed from R7; footprint Capacitor_SMD:C_0402_1005Metric_Pad0.74x0.62mm_HandSolder -> Resistor_SMD:R_0402_1005Metric
- renumbered C12 to C28, C13 to C29, C14 to C30, C15 to C31, J1 to J4, J2 to J5, R8 to R18, U4 to U7
Connections:
- net +3V3: now also FB2.2
- net at C32.1, C33.1, U7.1 (VCC_IN): now also FB2.1
