File: atlas-flight-controller-board-v4/stm32.kicad_sch (KiCad schematic)
At the start: 55 parts, among them J6 DX07S016JA1R1500, J7 Conn_01x08, J8 SWD_TC2030-NL, Q1 BSS138, SW2 SW_SPDT, SW3 SW_Push, U12 USBLC6, U13 STM32F405RGTx, Y1 16 MHz

Commit message: progress update. schematic has been done, layout is half finished. board is now 50x65mm for rf performance reasons
Parts:
- removed C38, C39, C40, C41, C42: 100 nF, Resistor_SMD:R_0402_1005Metric, symbol Device:C_Small
- removed C44, C45: 1 uF, Capacitor_SMD:C_0603_1608Metric, symbol Device:C_Small
- added C3, C4, C5, C6: 100n, Capacitor_SMD:C_0402_1005Metric, symbol Device:C_Small
- C10: renamed from C46; footprint Resistor_SMD:R_0402_1005Metric -> Capacitor_SMD:C_0402_1005Metric
- C11: renamed from C47; value 10 pF -> 10p; footprint Resistor_SMD:R_0402_1005Metric -> Capacitor_SMD:C_0402_1005Metric
- C12: renamed from C48; value 10 pF -> 10p; footprint Resistor_SMD:R_0402_1005Metric -> Capacitor_SMD:C_0402_1005Metric
- C15: renamed from C51; value 100 uF -> 100n
- C16: renamed from C52; value 100nF -> 100n
- C7: renamed from C43; value 10 nF -> 100n; footprint Capacitor_SMD:C_0603_1608Metric -> Capacitor_SMD:C_0402_1005Metric
- FB1: renamed from FB4; footprint (none) -> Inductor_SMD:L_0402_1005Metric
- SW1: renamed from SW2; footprint (none) -> Button_Switch_SMD:Nidec_Copal_CAS-120A
- renumbered C37 to C1, C49 to C13, C50 to C14, D4 to D1, D5 to D2, D6 to D3, D7 to D4, J6 to J1, J7 to J2, J8 to J3, R24 to R1, R33 to R10, R25 to R2, R26 to R3, R27 to R4, R28 to R5, R29 to R6, R30 to R7, R31 to R8, R32 to R9, SW3 to SW2, U12 to U1, U13 to U2, U14 to U3
Connections:
- net +3V3: now also C3.1, C4.1, C5.1, C6.1
- net GND: now also SW2.1, C3.2, C4.2, C5.2, C6.2; no longer SW2.2
- net PYRO_SEL0: now also U2.57 (PB5); no longer U2.62 (PB9)
- net PYRO_SEL1: now also U2.62 (PB9); no longer U2.57 (PB5)
- net at C16.2, R10.2: now also SW2.2; no longer SW2.1
Other:
- moved on the sheet: C10, FB1
